Commit message: Initial commit

File: vawt_ws/src/vawt_1/urdf/macros/blade_w_struts.xacro (robot description, xacro)
@@ -42,4 +42,14 @@
       <limit effort="300" velocity="0.1" lower="-3.14" upper="3.14"/>
     </joint>
+    <transmission name="${blade_name}_transmission">
+      <type>transmission_interface/SimpleTransmission</type>
+      <joint name="${blade_name}_joint">
+        <hardwareInterface>hardware_interface/EffortJointInterface</hardwareInterface>
+      </joint>
+      <actuator name="${blade_name}_motor">
+        <hardwareInterface>EffortJointInterface</hardwareInterface>
+        <mechanicalReduction>1</mechanicalReduction>
+      </actuator>
+    </transmission>
     <xacro:box_link link_name="${blade_name}" width="${blade_width}" height="${blade_height}" depth="${blade_depth}"
       xyz="0 0 ${blade_depth/6}" rpy="0 0 ${pi/2}" material="green" mass="${mass}"/>

File: vawt_ws/src/vawt_1/urdf/minimal/vawt_1.xacro (robot description, xacro)
@@ -28,16 +28,6 @@
     <origin xyz="0 0 ${base_depth + 0.01}"/>
     <axis xyz="0 0 1" />
-    <dynamics damping="0.2" friction="1"/>
+    <dynamics damping="0" friction="1"/>
   </joint>
-  <!-- transmission -->
-  <transmission name="main_shaft_joint_trans">
-    <type>transmission_interface/SimpleTransmission</type>
-    <actuator name="main_shaft_motor">
-      <mechanicalReduction>1</mechanicalReduction>
-    </actuator>
-    <joint name="main_shaft_joint">
-      <hardwareInterface>hardware_interface/EffortJointInterface</hardwareInterface>
-    </joint>
-  </transmission>
   <!-- main_shaft Link -->
   <xacro:property name="ms_radius" value="0.1" /> <!-- r  -->
@@ -46,9 +36,3 @@
   <xacro:cylinder_link link_name="${shaft_name}" length="${ms_length}" radius="${ms_radius}"
     xyz="0 0 ${ms_length/2}" rpy="0 0 0" material="blue" mass="${mass}"/>
-  <!-- blade_1  -->
-  <xacro:blade_w_struts blade_name="blade_1" parent_name="${shaft_name}" shaft_radius="${ms_radius}"
-    shaft_length="${ms_length}" blade_offset="0"/>
-  <!-- blade_2  -->
-  <xacro:blade_w_struts blade_name="blade_2" parent_name="${shaft_name}" shaft_radius="${ms_radius}"
-    shaft_length="${ms_length}" blade_offset="${pi}"/>
 </robot>

File: vawt_ws/src/vawt_1/urdf/oryg/vawt_1.xacro (robot description, xacro)
@@ -28,16 +28,6 @@
     <origin xyz="0 0 ${base_depth + 0.01}"/>
     <axis xyz="0 0 1" />
-    <dynamics damping="0.2" friction="1"/>
+    <dynamics damping="0" friction="1"/>
   </joint>
-  <!-- transmission -->
-  <transmission name="main_shaft_joint_trans">
-    <type>transmission_interface/SimpleTransmission</type>
-    <actuator name="main_shaft_motor">
-      <mechanicalReduction>1</mechanicalReduction>
-    </actuator>
-    <joint name="main_shaft_joint">
-      <hardwareInterface>hardware_interface/EffortJointInterface</hardwareInterface>
-    </joint>
-  </transmission>
   <!-- main_shaft Link -->
   <xacro:property name="ms_radius" value="0.1" /> <!-- r  -->

Commit message: physical model added joint_states subscriber added blade command publishers

File: vawt_ws/src/vawt_1/urdf/macros/blade_w_struts.xacro (robot description, xacro)
@@ -40,13 +40,13 @@
       <origin xyz="${shaft_radius + strut_depth} 0 0" rpy="0 0 0"/>
       <axis xyz="0 0 1" />
-      <limit effort="300" velocity="0.1" lower="-3.14" upper="3.14"/>
+      <limit effort="300" velocity="200" lower="-3.14" upper="3.14"/>
     </joint>
     <transmission name="${blade_name}_transmission">
       <type>transmission_interface/SimpleTransmission</type>
       <joint name="${blade_name}_joint">
-        <hardwareInterface>hardware_interface/EffortJointInterface</hardwareInterface>
+        <hardwareInterface>hardware_interface/PositionJointInterface</hardwareInterface>
       </joint>
       <actuator name="${blade_name}_motor">
-        <hardwareInterface>EffortJointInterface</hardwareInterface>
+        <hardwareInterface>PositionJointInterface</hardwareInterface>
         <mechanicalReduction>1</mechanicalReduction>
       </actuator>

Commit message: made 4d interpolation for getting optimal path

File: vawt_ws/src/vawt_1/urdf/macros/blade_w_struts.xacro (robot description, xacro)
@@ -40,5 +40,5 @@
       <origin xyz="${shaft_radius + strut_depth} 0 0" rpy="0 0 0"/>
       <axis xyz="0 0 1" />
-      <limit effort="300" velocity="200" lower="-3.14" upper="3.14"/>
+      <limit effort="300" velocity="100" lower="-1.3" upper="1.3"/>
     </joint>
     <transmission name="${blade_name}_transmission">

Commit message: ros hardware interface boilerplate

File: vawt_ws/src/vawt_1/urdf/macros/blade_w_struts.xacro (robot description, xacro)
@@ -48,5 +48,5 @@
       </joint>
       <actuator name="${blade_name}_motor">
-        <hardwareInterface>PositionJointInterface</hardwareInterface>
+        <hardwareInterface>hardware_interface/PositionJointInterface</hardwareInterface>
         <mechanicalReduction>1</mechanicalReduction>
       </actuator>

File: vawt_ws/src/vawt_1/urdf/vawt_1.xacro (robot description, xacro)
@@ -33,10 +33,11 @@
   <transmission name="main_shaft_joint_trans">
     <type>transmission_interface/SimpleTransmission</type>
+    <joint name="main_shaft_joint">
+      <hardwareInterface>hardware_interface/PositionJointInterface</hardwareInterface>
+    </joint>
     <actuator name="main_shaft_motor">
-      <mechanicalReduction>1</mechanicalReduction>
+        <hardwareInterface>hardware_interface/PositionJointInterface</hardwareInterface>
+        <mechanicalReduction>1</mechanicalReduction>
     </actuator>
-    <joint name="main_shaft_joint">
-      <hardwareInterface>hardware_interface/EffortJointInterface</hardwareInterface>
-    </joint>
   </transmission>
   <!-- main_shaft Link -->
